File: STM32.kicad_sch (KiCad schematic)
At the start: 41 parts

Commit message: update
Parts:
- removed C? (x2): 2u2, symbol Device:C_Small
- removed C?: 10n, symbol Device:C
- removed C?: 1u, symbol Device:C
- removed C? (x5): 100n, symbol Device:C
- removed C?: 4u7, symbol Device:C
- added C? (x7): 100n, symbol Device:C_Small
- added C?: 4u7, symbol Device:C_Small
- added C? (x2): 10n, symbol Device:C_Small
- added C? (x3): 2u2, symbol Device:C_Small
- added C?: 1u, symbol Device:C_Small
- added R? (x4): 2u2, symbol Device:R_Small
- added U?: MPU-6050, Sensor_Motion:InvenSense_QFN-24_4x4mm_P0.5mm, symbol Sensor_Motion:MPU-6050
- R?: value 15k -> 22
Connections:
- net +3.3V: now also C?.1, C?.1, C?.1, C?.1, C?.1, C?.1, C?.1, C?.1, C?.1, C?.2, R?.2, R?.2, R?.2, R?.2, U?.13 (VDD), U?.8 (VDDIO)
- net GND: now also C?.1, C?.2, C?.2, C?.2, C?.2, C?.2, C?.2, C?.2, C?.2, C?.2, C?.2, C?.2, C?.2, C?.2, U?.1 (CLKIN), U?.11 (FSYNC), U?.18 (GND), U?.9 (AD0)
- net I2C1_SCL: now also R?.1, U?.23 (SCL)
- net I2C1_SDA: now also R?.1, U?.24 (SDA)
- net I2C2_SCL: now also R?.1
- net I2C2_SDA: now also R?.1
- net at U?.31 (VCAP_1): now also C?.1
- net at U?.47 (VCAP_2): now also C?.1
- net IMU_IINT: now reaches U?.57 (PB5)
- net IMU_IINT: now also U?.12 (INT)
- new net: C?.1, U?.10 (REGOUT)
- new net: C?.1, U?.20 (CPOUT)
- no-connect marks 42 -> 43

Commit message: update
Parts:
- added C?: 100n, symbol Device:C_Small
- added J?: Conn_01x06, symbol Connector_Generic:Conn_01x06
- added J?: Conn_01x12, symbol Connector_Generic:Conn_01x12
- added R? (x3): 22, symbol Device:R_Small
Connections:
- net +3.3V: now also J?.12 (Pin_12), J?.6 (Pin_6)
- net GND: now also C?.2, J?.11 (Pin_11), J?.5 (Pin_5)
- net NRST: now also C?.1, R?.1; no longer J?.10 (Pin_10)
- net SWCLK: now also R?.1; no longer J?.4 (Pin_4)
- net SWO: now also R?.1; no longer J?.6 (Pin_6)
- net GPIO_AN1: now reaches U?.21 (PA5)
- net GPIO_AN1: now also J?.1 (Pin_1)
- net GPIO_AN2: now reaches U?.22 (PA6)
- net GPIO_AN2: now also J?.2 (Pin_2)
- net GPIO_AN3: now reaches U?.23 (PA7)
- net GPIO_AN3: now also J?.3 (Pin_3)
- net GPIO_AN4: now reaches U?.24 (PC4)
- net GPIO_AN4: now also J?.4 (Pin_4)
- net GPIO_OUT5: now reaches U?.33 (PB12)
- net GPIO_OUT5: now also J?.10 (Pin_10)
- net GPIO_OUT4: now reaches U?.34 (PB13)
- net GPIO_OUT4: now also J?.9 (Pin_9)
- net GPIO_OUT3: now reaches U?.35 (PB14)
- net GPIO_OUT3: now also J?.8 (Pin_8)
- net GPIO_OUT2: now reaches U?.36 (PB15)
- net GPIO_OUT2: now also J?.7 (Pin_7)
- net GPIO_OUT1: now reaches U?.37 (PC6)
- net GPIO_OUT1: now also J?.6 (Pin_6)
- net GPIO_IN5: now reaches U?.38 (PC7)
- net GPIO_IN5: now also J?.5 (Pin_5)
- net GPIO_IN4: now reaches U?.39 (PC8)
- net GPIO_IN4: now also J?.4 (Pin_4)
- net GPIO_IN3: now reaches U?.40 (PC9)
- net GPIO_IN3: now also J?.3 (Pin_3)
- net GPIO_IN2: now reaches U?.41 (PA8)
- net GPIO_IN2: now also J?.2 (Pin_2)
- net GPIO_IN1: now reaches U?.42 (PA9)
- net GPIO_IN1: now also J?.1 (Pin_1)
- new net: J?.10 (Pin_10), R?.2
- new net: J?.4 (Pin_4), R?.2
- new net: J?.6 (Pin_6), R?.2
- no-connect marks 43 -> 29
Other:
- moved on the sheet: C?, J?, R?, U?
