File: STM32/STM32.kicad_pcb (KiCad board)
At the start: 4 copper layers, 62 parts, among them J1 Screw_Terminal_01x02, J2 Conn_01x12, J3 USB_B_Micro, J4 SWD, J5 Conn_01x06, J6 Conn_01x04, J7 Conn_01x04, Q1 AO3401A, SW1 SW_SPDT, U1 MP2359DJ-LF-Z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

Commit message: pc
Parts:
- removed F1: 250mA, Fuse:Fuse_1206_3216Metric
- added D4: Red, LED_SMD:LED_0603_1608Metric, F.Cu at (73.7, 106.7)
- added F2: 250mA, Fuse:Fuse_1206_3216Metric, F.Cu at (116.8, 100.8)
- added R17: 1k, Resistor_SMD:R_0603_1608Metric, F.Cu at (77.7, 106.6)
- J4: footprint Connector_PinSocket_1.27mm:PinSocket_2x04_P1.27mm_Vertical_SMD -> Connector_PinSocket_1.27mm:PinSocket_2x05_P1.27mm_Vertical_SMD
- R2, R3, R4, R5: footprint Resistor_SMD:R_0201_0603Metric -> Resistor_SMD:R_0603_1608Metric
- moved C14 110.1 mm to (77.7, 97.2), turned to 180 degrees
- moved R14 99.9 mm to (73.3, 112.9), turned to 180 degrees
- moved C7 97.4 mm to (76.2, 86.2), turned to -90 degrees
- moved L2 95.0 mm to (78.2, 101.6), turned to 180 degrees
- moved C19 92.2 mm to (80.7, 98.3), turned to 90 degrees
- moved J1 91.7 mm to (134.6, 97.2), turned to 90 degrees
- moved C15 89.6 mm to (94.6, 102.9)
- moved C6 84.9 mm to (79.5, 89.9), turned to 180 degrees
- moved R8 83.5 mm to (93.9, 89.9), turned to 90 degrees
- moved R10 79.2 mm to (86.3, 88.3), turned to -90 degrees
- moved C21 76.7 mm to (80.8, 96.5), turned to 180 degrees
- moved C11 75.8 mm to (84.6, 89.2)
- moved C18 75.7 mm to (78.2, 100.3)
- moved Crystal1 75.7 mm to (77.7, 94.2), turned to -90 degrees
- moved C20 74.5 mm to (79.3, 98.3), turned to 90 degrees
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Connections:
- FB1 pad 2: Net-(D1-Pad1) -> Net-(F2-Pad2)
- J7 pad 2: I2C1_SDA -> I2C2_SDA
- J7 pad 3: I2C1_SCL -> I2C2_SCL
- Q1 pad 3: Net-(F1-Pad2) -> +12V
Routing:
- net GND: track 0.00 -> 126.1 mm, vias 0 -> 46
- net +3.3V: track 0.00 -> 87.3 mm, vias 0 -> 40
- net GPIO_IN1: track 0.00 -> 42.0 mm
- net GPIO_IN2: track 0.00 -> 40.3 mm
- net GPIO_IN4: track 0.00 -> 39.2 mm, vias 0 -> 2
- net GPIO_IN3: track 0.00 -> 38.6 mm
- net Net-(J4-Pad2): track 0.00 -> 37.7 mm
- net USB_D-: track 0.00 -> 37.3 mm
- net USB_D+: track 0.00 -> 37.3 mm
- net Net-(J4-Pad6): track 0.00 -> 35.6 mm, vias 0 -> 2
- net +5V: track 0.00 -> 32.1 mm
- net Net-(J4-Pad4): track 0.00 -> 31.5 mm, vias 0 -> 2
- net GPIO_IN5: track 0.00 -> 30.2 mm
- net GPIO_OUT1: track 0.00 -> 27.7 mm
- net I2C2_SDA: track 0.00 -> 27.5 mm, vias 0 -> 2
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- added copper zone on In2.Cu, net +3.3V
- added copper zone on In1.Cu, net GND
Other:
- board outline added: 81.3 x 50.8 mm

Commit message: pc
Parts:
- added G***: LOGO, Kronos:logo, F.Cu at (67.3, 94.0)
- moved SW1 1.34 mm to (86.2, 74.9)
Routing:
- net unconnected-(J3-Pad6): track 0.00 -> 12.6 mm, vias 0 -> 2
- net /SW_BOOT: track 18.1 -> 16.8 mm
Other:
- outline, holes or cut-outs redrawn
- board text added: "+"
- board text added: "+12V"
- board text added: "+3.3"
- board text added: "AN1"
- board text added: "AN2"
- board text added: "AN3"
- board text added: "AN4"
- board text added: "BOOT"
- board text added: "GND"
- board text added: "I2C"
- board text added: "IN1"
- board text added: "IN2"
- board text added: "IN3"
- board text added: "IN4"
- board text added: "IN5"
- board text added: "JLCJLCJLCJLC"
- board text added: "N. P."
- board text added: "OUT1"
- board text added: "OUT2"
- board text added: "OUT3"
- board text added: "OUT4"
- board text added: "OUT5"
- board text added: "PREDEEP BALASUBRAMANIAN"
- board text added: "RUN"
- board text added: "SCL"
- board text added: "SDA"
- board text added: "UART"
- board text added: "USB"
