File: STM32/STM32.kicad_sch (KiCad schematic)
At the start: 62 parts, among them J1 Screw_Terminal_01x02, J2 Conn_01x12, J3 USB_B_Micro, J4 SWD, J5 Conn_01x06, J6 Conn_01x04, J7 Conn_01x04, Q1 AO3401A, SW1 SW_SPDT, U1 MP2359DJ-LF-Z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

Commit message: pc
Parts:
- removed F1: 250mA, Fuse:Fuse_1206_3216Metric, symbol Device:Polyfuse_Small
- added D4: Red, LED_SMD:LED_0603_1608Metric, symbol Device:LED_Small
- added F2: 250mA, Fuse:Fuse_1206_3216Metric, symbol Device:Polyfuse_Small
- added R17: 1k, Resistor_SMD:R_0603_1608Metric, symbol Device:R_Small
- J4: footprint Connector_PinSocket_1.27mm:PinSocket_2x04_P1.27mm_Vertical_SMD -> Connector_PinSocket_1.27mm:PinSocket_2x05_P1.27mm_Vertical_SMD
- R2, R3, R4, R5: footprint Resistor_SMD:R_0201_0603Metric -> Resistor_SMD:R_0603_1608Metric
Connections:
- net +12V: now also Q1.3 (D)
- net +3.3V: now also D4.2 (A)
- net GND: now also R17.2
- net I2C1_SCL: no longer J7.3 (Pin_3)
- net I2C1_SDA: no longer J7.2 (Pin_2)
- net I2C2_SCL: now also J7.3 (Pin_3)
- net I2C2_SDA: now also J7.2 (Pin_2)
- net at D1.1 (K), Q1.2 (S): now also F2.1; no longer FB1.2
- new net: F2.2, FB1.2
- new net: D4.1 (K), R17.1
Other:
- moved on the sheet: C1, C3, FB1, R4, R5

Commit message: pc
Parts:
- C1, C2, C4: LCSC Part # (none) -> C1954312
- C10, C14: LCSC Part # (none) -> C3876622
- C11, C12, C15, C17, C18, C21, C6, C7: LCSC Part # (none) -> C361203
- C13, C16, C8: LCSC Part # (none) -> C1953313
- C19: LCSC Part # (none) -> C386111
- C20: LCSC Part # (none) -> C1954072
- C3: LCSC Part # (none) -> C77497
- C5: LCSC Part # (none) -> C2835533
- C9: LCSC Part # (none) -> C2844393
- Crystal1: LCSC Part # (none) -> C160456
- D1, D2: LCSC Part # (none) -> C779771
- D3: LCSC Part # (none) -> C3148192
- D4: LCSC Part # (none) -> C84263
- F2: LCSC Part # (none) -> C369159
- FB1: LCSC Part # (none) -> C1017
- L1: LCSC Part # (none) -> C139506
- L2: LCSC Part # (none) -> C26443
- Q1: LCSC Part # (none) -> C306862
- R1: LCSC Part # (none) -> C227501
- R10: LCSC Part # (none) -> C328298
- R11, R17: LCSC Part # (none) -> C269704
- R12, R13, R14, R15: LCSC Part # (none) -> C3017487
- R16: LCSC Part # (none) -> C1096
- R2: LCSC Part # (none) -> C3152125
- R3: LCSC Part # (none) -> C667461
- R4: LCSC Part # (none) -> C667752
- R5: LCSC Part # (none) -> C912142
- R6, R7, R8, R9: LCSC Part # (none) -> C174144
- U1: LCSC Part # (none) -> C14259
- U3: LCSC Part # (none) -> C24112
- U4: LCSC Part # (none) -> C15742

Commit message: pc
Parts:
- C10, C14: LCSC Part # C3876622 -> C76700
- C20: LCSC Part # C1954072 -> C913556
- D3: LCSC Part # C3148192 -> C397049
- D4: LCSC Part # C84263 -> C90692
- L1: LCSC Part # C139506 -> C150031
Changed lines of the file:
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@@
       (effects (font (size 1.27 1.27)) hide)
     )
-    (property "LCSC Part #" "C3876622" (id 4) (at 264.16 218.44 0)
+    (property "LCSC Part #" "C76700" (id 4) (at 264.16 218.44 0)
       (effects (font (size 1.27 1.27)) hide)
     )
@@
       (effects (font (size 1.27 1.27)) hide)
     )
-    (property "LCSC Part #" "C3148192" (id 4) (at 383.54 229.87 0)
+    (property "LCSC Part #" "C397049" (id 4) (at 383.54 229.87 0)
       (effects (font (size 1.27 1.27)) hide)
     )
@@
       (effects (font (size 1.27 1.27)) hide)
     )
-    (property "LCSC Part #" "C139506" (id 4) (at 72.39 78.74 0)
+    (property "LCSC Part #" "C150031" (id 4) (at 72.39 78.74 0)
       (effects (font (size 1.27 1.27)) hide)
     )
@@
       (effects (font (size 1.27 1.27)) hide)
     )
-    (property "LCSC Part #" "C84263" (id 4) (at 262.89 254 0)
+    (property "LCSC Part #" "C90692" (id 4) (at 262.89 254 0)
       (effects (font (size 1.27 1.27)) hide)
     )
@@
       (effects (font (size 1.27 1.27)) hide)
     )
-    (property "LCSC Part #" "C1954072" (id 4) (at 356.87 140.97 0)
+    (property "LCSC Part #" "C913556" (id 4) (at 356.87 140.97 0)
       (effects (font (size 1.27 1.27)) hide)
     )
@@
       (effects (font (size 1.27 1.27)) hide)
     )
-    (property "LCSC Part #" "C3876622" (id 4) (at 287.02 218.44 0)
-      (effects (font (size 1.27 1.27)) hide)
-    )
+    (property "LCSC Part #" "C76700" (id 4) (at 287.02 218.44 0)
+      (effects (font (size 1.27 1.27)) hide)
+    )
